File: Hardware/mood/mood.kicad_sch (KiCad schematic)
At the start: 91 parts, among them IC1 ESP32-C3-WROOM-02-H4, IC2 TPS564247DRLR, IC6 SC810ULTRT, J1 Conn_02x03_Odd_Even, J2 USB_C_Receptacle_USB2.0, Q1 C347476, Q2 C347476, Q3 C347476, SW1 SW_SPST, SW2 SW_SPST

Commit message: Mood complete, working on fft webpage
Other:
- moved on the sheet: C2, C3, C4, C5, C7, C8, H1, H2, IC2, J1, L1, Q1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
